File: uProject.kicad_sch (KiCad schematic)
At the start: 10 parts, among them P1 HC-SR501, P2 HC-SR501, SW1 SW_DPST_x2, U1 AT89C51, U2 LCD-16X2, Y1 Crystal

Commit message: version2
Connections:
- net at P1.2 (DATA): now also U1.14 (P3.2/~{INT0}); no longer U1.2 (P1.0)
- net at U1.15 (P3.3/~{INT1}): now also P2.2 (DATA)
- net at U1.3 (P1.1): no longer P2.2 (DATA)
Changed lines of the file:
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@@
+	(wire
+		(pts
+			(xy 120.65 115.57) (xy 127 115.57)
+		)
+		(stroke
+			(width 0)
+			(type default)
+		)
+	)
 	(wire
 		(pts
@@
 	(wire
 		(pts
-			(xy 114.3 107.95) (xy 114.3 85.09)
-		)
-		(stroke
-			(width 0)
-			(type default)
-		)
-	)
-	(wire
-		(pts
 			(xy 167.64 100.33) (xy 177.8 100.33)
 		)
@@
 	(wire
 		(pts
-			(xy 92.71 107.95) (xy 114.3 107.95)
+			(xy 92.71 107.95) (xy 121.92 107.95)
 		)
 		(stroke
@@
 	(wire
 		(pts
-			(xy 120.65 87.63) (xy 127 87.63)
-		)
-		(stroke
-			(width 0)
-			(type default)
-		)
-	)
-	(wire
-		(pts
 			(xy 185.42 92.71) (xy 185.42 107.95)
 		)
@@
 	(wire
 		(pts
-			(xy 120.65 130.81) (xy 120.65 87.63)
-		)
-		(stroke
-			(width 0)
-			(type default)
-		)
-	)
-	(wire
-		(pts
 			(xy 167.64 95.25) (xy 182.88 95.25)
 		)
@@
 	(wire
 		(pts
+			(xy 120.65 130.81) (xy 120.65 115.57)
+		)
+		(stroke
+			(width 0)
+			(type default)
+		)
+	)
+	(wire
+		(pts
 			(xy 167.64 90.17) (xy 187.96 90.17)
 		)
@@
 	(wire
 		(pts
+			(xy 121.92 107.95) (xy 121.92 113.03)
+		)
+		(stroke
+			(width 0)
+			(type default)
+		)
+	)
+	(wire
+		(pts
 			(xy 85.09 99.06) (xy 85.09 100.33)
 		)
@@
 	(wire
 		(pts
-			(xy 114.3 85.09) (xy 127 85.09)
-		)
-		(stroke
+			(xy 121.92 113.03) (xy 127 113.03)
+		)
+		(stroke
